Commit message: extended user plane

File: src/myur5sim/myur5_description/urdf/myur5.urdf.xacro (robot description, xacro)
@@ -52,5 +52,6 @@
         <origin xyz="0 0 0.05" rpy="0 0 0" />
         <geometry>
-            <box size="0.07 0.07 0.10"/>
+            <!--box size="0.07 0.07 0.10"/-->
+            <sphere radius ="0.04"/>
         </geometry>
         <material name="LightGrey">
@@ -61,5 +62,6 @@
         <origin xyz="0 0 0.05" rpy="0 0 0"/>
         <geometry>
-              <box size="0.07 0.07 0.10"/>
+              <!--box size="0.07 0.07 0.10"/-->
+              <sphere radius ="0.04"/>
         </geometry>
       </collision>
